File: pcb/kicad/left/left.sch (KiCad schematic (older format))
At the start: 61 parts, among them J1 USB_C_Receptacle_USB2.0, J2 AudioJack4, J3 Conn_01x12_Male, SW1 BOOT, SW10 SW_Push, SW12 SW_Push, SW13 SW_Push, SW14 SW_Push, SW15 SW_Push, SW17 SW_Push, SW18 SW_Push, SW19 SW_Push, SW2 RESET, SW21 SW_Push, SW22 SW_Push, SW23 SW_Push, SW24 SW_Push, SW3 SW_Push, SW31 SW_Push, SW32 SW_Push, SW33 SW_Push, SW34 SW_Push, SW4 SW_Push, SW5 SW_Push, SW7 SW_Push, SW8 SW_Push, SW9 SW_Push, U1 STM32, U2 LDO

Commit message: right advances
Parts:
- J3: footprint kicad-usb:Harwin_M20-89012xx_1x12_P2.54mm_Horizontal -> kicad-harwin:Harwin_M20-89012xx_1x12_P2.54mm_Horizontal
Connections:
- net GND: now also U1.25 (PB12)
Changed lines of the file:
@@
 EESchema Schematic File Version 4
-LIBS:keyboard-cache
 EELAYER 26 0
 EELAYER END
@@
 F 0 "J3" H 7473 2173 50  0000 R CNN
 F 1 "Conn_01x12_Male" H 7473 2082 50  0000 R CNN
-F 2 "kicad-usb:Harwin_M20-89012xx_1x12_P2.54mm_Horizontal" H 7500 2200 50  0001 C CNN
+F 2 "kicad-harwin:Harwin_M20-89012xx_1x12_P2.54mm_Horizontal" H 7500 2200 50  0001 C CNN
 F 3 "~" H 7500 2200 50  0001 C CNN
 	1    7500 2200
@@
 Text GLabel 6700 3000 2    50   Input ~ 0
 PA5
+$Comp
+L power:GND #PWR?
+U 1 1 5F02320E
+P 5400 3700
+F 0 "#PWR?" H 5400 3450 50  0001 C CNN
+F 1 "GND" V 5405 3572 50  0000 R CNN
+F 2 "" H 5400 3700 50  0001 C CNN
+F 3 "" H 5400 3700 50  0001 C CNN
+	1    5400 3700
+	0    1    1    0
+$EndComp
 $EndSCHEMATC

Commit message: left: correct diode bug
Parts:
- D10, D11, D12, D14, D15, D16, D17, D19, D20, D21, D23, D24, D25, D26, D33, D34, D35, D36, D5, D6, D7, D9: symbol pspice:DIODE -> Diode:1N4148WS
- J2: footprint Keebio:TRRS-PJ-320A-no-Fmask -> keebio:TRRS-PJ-320A-no-Fmask
Connections:
- net ROW1: now also D14.2 (A), D19.2 (A), D23.2 (A), D33.2 (A), D5.2 (A), D9.2 (A); no longer D14.1 (K), D19.1 (K), D23.1 (K), D33.1 (K), D5.1 (K), D9.1 (K)
- net ROW2: now also D10.2 (A), D15.2 (A), D20.2 (A), D24.2 (A), D34.2 (A), D6.2 (A); no longer D10.1 (K), D15.1 (K), D20.1 (K), D24.1 (K), D34.1 (K), D6.1 (K)
- net ROW3: now also D11.2 (A), D16.2 (A), D21.2 (A), D25.2 (A), D35.2 (A), D7.2 (A); no longer D11.1 (K), D16.1 (K), D21.1 (K), D25.1 (K), D35.1 (K), D7.1 (K)
- net ROW4: now also D12.2 (A), D17.2 (A), D26.2 (A), D36.2 (A); no longer D12.1 (K), D17.1 (K), D26.1 (K), D36.1 (K)
- net at SW9.1: now also D11.1 (K); no longer D11.2 (A)
- net at SW10.1: now also D12.1 (K); no longer D12.2 (A)
- net at SW8.1: now also D10.1 (K); no longer D10.2 (A)
- net at SW7.1: now also D9.1 (K); no longer D9.2 (A)
- net at SW23.1: now also D25.1 (K); no longer D25.2 (A)
- net at SW24.1: now also D26.1 (K); no longer D26.2 (A)
- net at SW22.1: now also D24.1 (K); no longer D24.2 (A)
- net at SW21.1: now also D23.1 (K); no longer D23.2 (A)
- net at SW33.1: now also D35.1 (K); no longer D35.2 (A)
- net at SW34.1: now also D36.1 (K); no longer D36.2 (A)
- net at SW32.1: now also D34.1 (K); no longer D34.2 (A)
- net at SW31.1: now also D33.1 (K); no longer D33.2 (A)
- net at SW5.1: now also D7.1 (K); no longer D7.2 (A)
- net at SW4.1: now also D6.1 (K); no longer D6.2 (A)
- net at SW3.1: now also D5.1 (K); no longer D5.2 (A)
- net at SW19.1: now also D21.1 (K); no longer D21.2 (A)
- net at SW18.1: now also D20.1 (K); no longer D20.2 (A)
- net at SW17.1: now also D19.1 (K); no longer D19.2 (A)
- net at SW14.1: now also D16.1 (K); no longer D16.2 (A)
- net at SW15.1: now also D17.1 (K); no longer D17.2 (A)
- net at SW13.1: now also D15.1 (K); no longer D15.2 (A)
- net at SW12.1: now also D14.1 (K); no longer D14.2 (A)
Other:
- moved on the sheet: SW12, SW13, SW14, SW15

Commit message: left: change switch footprint
Parts:
- SW10, SW12, SW13, SW14, SW15, SW17, SW18, SW19, SW21, SW22, SW23, SW24, SW3, SW31, SW32, SW33, SW34, SW4, SW5, SW7, SW8, SW9: footprint Keebio:MX-Alps-Choc-1U-NoLED -> foostan-kbd:CherryMX_Choc_1u
Changed lines of the file:
@@
 F 0 "SW9" H 1350 3635 50  0000 C CNN
 F 1 "SW_Push" H 1350 3544 50  0000 C CNN
-F 2 "Keebio:MX-Alps-Choc-1U-NoLED" H 1350 3550 50  0001 C CNN
+F 2 "foostan-kbd:CherryMX_Choc_1u" H 1350 3550 50  0001 C CNN
 F 3 "" H 1350 3550 50  0001 C CNN
 	1    1350 3350
@@
 F 0 "SW10" H 1350 4035 50  0000 C CNN
 F 1 "SW_Push" H 1350 3944 50  0000 C CNN
-F 2 "Keebio:MX-Alps-Choc-1U-NoLED" H 1350 3950 50  0001 C CNN
+F 2 "foostan-kbd:CherryMX_Choc_1u" H 1350 3950 50  0001 C CNN
 F 3 "" H 1350 3950 50  0001 C CNN
 	1    1350 3750
@@
 F 0 "SW8" H 1350 3235 50  0000 C CNN
 F 1 "SW_Push" H 1350 3144 50  0000 C CNN
-F 2 "Keebio:MX-Alps-Choc-1U-NoLED" H 1350 3150 50  0001 C CNN
+F 2 "foostan-kbd:CherryMX_Choc_1u" H 1350 3150 50  0001 C CNN
 F 3 "" H 1350 3150 50  0001 C CNN
 	1    1350 2950
@@
 F 0 "SW7" H 1350 2835 50  0000 C CNN
 F 1 "SW_Push" H 1350 2744 50  0000 C CNN
-F 2 "Keebio:MX-Alps-Choc-1U-NoLED" H 1350 2750 50  0001 C CNN
+F 2 "foostan-kbd:CherryMX_Choc_1u" H 1350 2750 50  0001 C CNN
 F 3 "" H 1350 2750 50  0001 C CNN
 	1    1350 2550
@@
 F 0 "SW23" H 2700 3635 50  0000 C CNN
 F 1 "SW_Push" H 2700 3544 50  0000 C CNN
-F 2 "Keebio:MX-Alps-Choc-1U-NoLED" H 2700 3550 50  0001 C CNN
+F 2 "foostan-kbd:CherryMX_Choc_1u" H 2700 3550 50  0001 C CNN
 F 3 "" H 2700 3550 50  0001 C CNN
 	1    2700 3350
@@
 F 0 "SW24" H 2700 4035 50  0000 C CNN
 F 1 "SW_Push" H 2700 3944 50  0000 C CNN
-F 2 "Keebio:MX-Alps-Choc-1U-NoLED" H 2700 3950 50  0001 C CNN
+F 2 "foostan-kbd:CherryMX_Choc_1u" H 2700 3950 50  0001 C CNN
 F 3 "" H 2700 3950 50  0001 C CNN
 	1    2700 3750
@@
 F 0 "SW22" H 2700 3235 50  0000 C CNN
 F 1 "SW_Push" H 2700 3144 50  0000 C CNN
-F 2 "Keebio:MX-Alps-Choc-1U-NoLED" H 2700 3150 50  0001 C CNN
+F 2 "foostan-kbd:CherryMX_Choc_1u" H 2700 3150 50  0001 C CNN
 F 3 "" H 2700 3150 50  0001 C CNN
 	1    2700 2950
@@
 F 0 "SW21" H 2700 2835 50  0000 C CNN
 F 1 "SW_Push" H 2700 2744 50  0000 C CNN
-F 2 "Keebio:MX-Alps-Choc-1U-NoLED" H 2700 2750 50  0001 C CNN
+F 2 "foostan-kbd:CherryMX_Choc_1u" H 2700 2750 50  0001 C CNN
 F 3 "" H 2700 2750 50  0001 C CNN
 	1    2700 2550
@@
 F 0 "SW33" H 4050 3635 50  0000 C CNN
 F 1 "SW_Push" H 4050 3544 50  0000 C CNN
-F 2 "Keebio:MX-Alps-Choc-1U-NoLED" H 4050 3550 50  0001 C CNN
+F 2 "foostan-kbd:CherryMX_Choc_1u" H 4050 3550 50  0001 C CNN
 F 3 "" H 4050 3550 50  0001 C CNN
 	1    4050 3350
@@
 F 0 "SW34" H 4050 4035 50  0000 C CNN
 F 1 "SW_Push" H 4050 3944 50  0000 C CNN
-F 2 "Keebio:MX-Alps-Choc-1U-NoLED" H 4050 3950 50  0001 C CNN
+F 2 "foostan-kbd:CherryMX_Choc_1u" H 4050 3950 50  0001 C CNN
 F 3 "" H 4050 3950 50  0001 C CNN
 	1    4050 3750
@@
 F 0 "SW32" H 4050 3235 50  0000 C CNN
 F 1 "SW_Push" H 4050 3144 50  0000 C CNN
-F 2 "Keebio:MX-Alps-Choc-1U-NoLED" H 4050 3150 50  0001 C CNN
+F 2 "foostan-kbd:CherryMX_Choc_1u" H 4050 3150 50  0001 C CNN
 F 3 "" H 4050 3150 50  0001 C CNN
 	1    4050 2950
@@
 F 0 "SW31" H 4050 2835 50  0000 C CNN
 F 1 "SW_Push" H 4050 2744 50  0000 C CNN
-F 2 "Keebio:MX-Alps-Choc-1U-NoLED" H 4050 2750 50  0001 C CNN
+F 2 "foostan-kbd:CherryMX_Choc_1u" H 4050 2750 50  0001 C CNN
 F 3 "" H 4050 2750 50  0001 C CNN
 	1    4050 2550
@@
 F 0 "SW5" H 1350 1935 50  0000 C CNN
 F 1 "SW_Push" H 1350 1844 50  0000 C CNN
-F 2 "Keebio:MX-Alps-Choc-1U-NoLED" H 1350 1850 50  0001 C CNN
+F 2 "foostan-kbd:CherryMX_Choc_1u" H 1350 1850 50  0001 C CNN
 F 3 "" H 1350 1850 50  0001 C CNN
 	1    1350 1650
@@
 F 0 "SW4" H 1350 1535 50  0000 C CNN
 F 1 "SW_Push" H 1350 1444 50  0000 C CNN
-F 2 "Keebio:MX-Alps-Choc-1U-NoLED" H 1350 1450 50  0001 C CNN
+F 2 "foostan-kbd:CherryMX_Choc_1u" H 1350 1450 50  0001 C CNN
 F 3 "" H 1350 1450 50  0001 C CNN
 	1    1350 1250
@@
 F 0 "SW3" H 1350 1135 50  0000 C CNN
 F 1 "SW_Push" H 1350 1044 50  0000 C CNN
-F 2 "Keebio:MX-Alps-Choc-1U-NoLED" H 1350 1050 50  0001 C CNN
+F 2 "foostan-kbd:CherryMX_Choc_1u" H 1350 1050 50  0001 C CNN
 F 3 "" H 1350 1050 50  0001 C CNN
 	1    1350 850
@@
 F 0 "SW19" H 2700 1935 50  0000 C CNN
 F 1 "SW_Push" H 2700 1844 50  0000 C CNN
-F 2 "Keebio:MX-Alps-Choc-1U-NoLED" H 2700 1850 50  0001 C CNN
+F 2 "foostan-kbd:CherryMX_Choc_1u" H 2700 1850 50  0001 C CNN
 F 3 "" H 2700 1850 50  0001 C CNN
 	1    2700 1650
@@
 F 0 "SW18" H 2700 1535 50  0000 C CNN
 F 1 "SW_Push" H 2700 1444 50  0000 C CNN
-F 2 "Keebio:MX-Alps-Choc-1U-NoLED" H 2700 1450 50  0001 C CNN
+F 2 "foostan-kbd:CherryMX_Choc_1u" H 2700 1450 50  0001 C CNN
 F 3 "" H 2700 1450 50  0001 C CNN
 	1    2700 1250
@@
 F 0 "SW17" H 2700 1135 50  0000 C CNN
 F 1 "SW_Push" H 2700 1044 50  0000 C CNN
-F 2 "Keebio:MX-Alps-Choc-1U-NoLED" H 2700 1050 50  0001 C CNN
+F 2 "foostan-kbd:CherryMX_Choc_1u" H 2700 1050 50  0001 C CNN
 F 3 "" H 2700 1050 50  0001 C CNN
 	1    2700 850
@@
 F 0 "SW14" H 1350 5585 50  0000 C CNN
 F 1 "SW_Push" H 1350 5494 50  0000 C CNN
-F 2 "Keebio:MX-Alps-Choc-1U-NoLED" H 1350 5500 50  0001 C CNN
+F 2 "foostan-kbd:CherryMX_Choc_1u" H 1350 5500 50  0001 C CNN
 F 3 "" H 1350 5500 50  0001 C CNN
 	1    1350 5300
@@
 F 0 "SW15" H 1350 5985 50  0000 C CNN
 F 1 "SW_Push" H 1350 5894 50  0000 C CNN
-F 2 "Keebio:MX-Alps-Choc-1U-NoLED" H 1350 5900 50  0001 C CNN
+F 2 "foostan-kbd:CherryMX_Choc_1u" H 1350 5900 50  0001 C CNN
 F 3 "" H 1350 5900 50  0001 C CNN
 	1    1350 5700
@@
 F 0 "SW13" H 1350 5185 50  0000 C CNN
 F 1 "SW_Push" H 1350 5094 50  0000 C CNN
-F 2 "Keebio:MX-Alps-Choc-1U-NoLED" H 1350 5100 50  0001 C CNN
+F 2 "foostan-kbd:CherryMX_Choc_1u" H 1350 5100 50  0001 C CNN
 F 3 "" H 1350 5100 50  0001 C CNN
 	1    1350 4900
@@
 F 0 "SW12" H 1350 4785 50  0000 C CNN
 F 1 "SW_Push" H 1350 4694 50  0000 C CNN
-F 2 "Keebio:MX-Alps-Choc-1U-NoLED" H 1350 4700 50  0001 C CNN
+F 2 "foostan-kbd:CherryMX_Choc_1u" H 1350 4700 50  0001 C CNN
 F 3 "" H 1350 4700 50  0001 C CNN
 	1    1350 4500
@@
 PA5
 $Comp
-L power:GND #PWR?
+L power:GND #PWR0110
 U 1 1 5F02320E
 P 5400 3700
-F 0 "#PWR?" H 5400 3450 50  0001 C CNN
+F 0 "#PWR0110" H 5400 3450 50  0001 C CNN
 F 1 "GND" V 5405 3572 50  0000 R CNN
 F 2 "" H 5400 3700 50  0001 C CNN

Commit message: custom switch footprint
Parts:
- SW10, SW12, SW13, SW14, SW15, SW17, SW18, SW19, SW21, SW22, SW23, SW24, SW3, SW31, SW32, SW33, SW34, SW4, SW5, SW7, SW8, SW9: footprint foostan-kbd:CherryMX_Choc_1u -> custom:CherryMX_Choc_1u
Changed lines of the file:
@@
 F 0 "SW9" H 1350 3635 50  0000 C CNN
 F 1 "SW_Push" H 1350 3544 50  0000 C CNN
-F 2 "foostan-kbd:CherryMX_Choc_1u" H 1350 3550 50  0001 C CNN
+F 2 "custom:CherryMX_Choc_1u" H 1350 3550 50  0001 C CNN
 F 3 "" H 1350 3550 50  0001 C CNN
 	1    1350 3350
@@
 F 0 "SW10" H 1350 4035 50  0000 C CNN
 F 1 "SW_Push" H 1350 3944 50  0000 C CNN
-F 2 "foostan-kbd:CherryMX_Choc_1u" H 1350 3950 50  0001 C CNN
+F 2 "custom:CherryMX_Choc_1u" H 1350 3950 50  0001 C CNN
 F 3 "" H 1350 3950 50  0001 C CNN
 	1    1350 3750
@@
 F 0 "SW8" H 1350 3235 50  0000 C CNN
 F 1 "SW_Push" H 1350 3144 50  0000 C CNN
-F 2 "foostan-kbd:CherryMX_Choc_1u" H 1350 3150 50  0001 C CNN
+F 2 "custom:CherryMX_Choc_1u" H 1350 3150 50  0001 C CNN
 F 3 "" H 1350 3150 50  0001 C CNN
 	1    1350 2950
@@
 F 0 "SW7" H 1350 2835 50  0000 C CNN
 F 1 "SW_Push" H 1350 2744 50  0000 C CNN
-F 2 "foostan-kbd:CherryMX_Choc_1u" H 1350 2750 50  0001 C CNN
+F 2 "custom:CherryMX_Choc_1u" H 1350 2750 50  0001 C CNN
 F 3 "" H 1350 2750 50  0001 C CNN
 	1    1350 2550
@@
 F 0 "SW23" H 2700 3635 50  0000 C CNN
 F 1 "SW_Push" H 2700 3544 50  0000 C CNN
-F 2 "foostan-kbd:CherryMX_Choc_1u" H 2700 3550 50  0001 C CNN
+F 2 "custom:CherryMX_Choc_1u" H 2700 3550 50  0001 C CNN
 F 3 "" H 2700 3550 50  0001 C CNN
 	1    2700 3350
@@
 F 0 "SW24" H 2700 4035 50  0000 C CNN
 F 1 "SW_Push" H 2700 3944 50  0000 C CNN
-F 2 "foostan-kbd:CherryMX_Choc_1u" H 2700 3950 50  0001 C CNN
+F 2 "custom:CherryMX_Choc_1u" H 2700 3950 50  0001 C CNN
 F 3 "" H 2700 3950 50  0001 C CNN
 	1    2700 3750
@@
 F 0 "SW22" H 2700 3235 50  0000 C CNN
 F 1 "SW_Push" H 2700 3144 50  0000 C CNN
-F 2 "foostan-kbd:CherryMX_Choc_1u" H 2700 3150 50  0001 C CNN
+F 2 "custom:CherryMX_Choc_1u" H 2700 3150 50  0001 C CNN
 F 3 "" H 2700 3150 50  0001 C CNN
 	1    2700 2950
@@
 F 0 "SW21" H 2700 2835 50  0000 C CNN
 F 1 "SW_Push" H 2700 2744 50  0000 C CNN
-F 2 "foostan-kbd:CherryMX_Choc_1u" H 2700 2750 50  0001 C CNN
+F 2 "custom:CherryMX_Choc_1u" H 2700 2750 50  0001 C CNN
 F 3 "" H 2700 2750 50  0001 C CNN
 	1    2700 2550
@@
 F 0 "SW33" H 4050 3635 50  0000 C CNN
 F 1 "SW_Push" H 4050 3544 50  0000 C CNN
-F 2 "foostan-kbd:CherryMX_Choc_1u" H 4050 3550 50  0001 C CNN
+F 2 "custom:CherryMX_Choc_1u" H 4050 3550 50  0001 C CNN
 F 3 "" H 4050 3550 50  0001 C CNN
 	1    4050 3350
@@
 F 0 "SW34" H 4050 4035 50  0000 C CNN
 F 1 "SW_Push" H 4050 3944 50  0000 C CNN
-F 2 "foostan-kbd:CherryMX_Choc_1u" H 4050 3950 50  0001 C CNN
+F 2 "custom:CherryMX_Choc_1u" H 4050 3950 50  0001 C CNN
 F 3 "" H 4050 3950 50  0001 C CNN
 	1    4050 3750
@@
 F 0 "SW32" H 4050 3235 50  0000 C CNN
 F 1 "SW_Push" H 4050 3144 50  0000 C CNN
-F 2 "foostan-kbd:CherryMX_Choc_1u" H 4050 3150 50  0001 C CNN
+F 2 "custom:CherryMX_Choc_1u" H 4050 3150 50  0001 C CNN
 F 3 "" H 4050 3150 50  0001 C CNN
 	1    4050 2950
@@
 F 0 "SW31" H 4050 2835 50  0000 C CNN
 F 1 "SW_Push" H 4050 2744 50  0000 C CNN
-F 2 "foostan-kbd:CherryMX_Choc_1u" H 4050 2750 50  0001 C CNN
+F 2 "custom:CherryMX_Choc_1u" H 4050 2750 50  0001 C CNN
 F 3 "" H 4050 2750 50  0001 C CNN
 	1    4050 2550
@@
 F 0 "SW5" H 1350 1935 50  0000 C CNN
 F 1 "SW_Push" H 1350 1844 50  0000 C CNN
-F 2 "foostan-kbd:CherryMX_Choc_1u" H 1350 1850 50  0001 C CNN
+F 2 "custom:CherryMX_Choc_1u" H 1350 1850 50  0001 C CNN
 F 3 "" H 1350 1850 50  0001 C CNN
 	1    1350 1650
@@
 F 0 "SW4" H 1350 1535 50  0000 C CNN
 F 1 "SW_Push" H 1350 1444 50  0000 C CNN
-F 2 "foostan-kbd:CherryMX_Choc_1u" H 1350 1450 50  0001 C CNN
+F 2 "custom:CherryMX_Choc_1u" H 1350 1450 50  0001 C CNN
 F 3 "" H 1350 1450 50  0001 C CNN
 	1    1350 1250
@@
 F 0 "SW3" H 1350 1135 50  0000 C CNN
 F 1 "SW_Push" H 1350 1044 50  0000 C CNN
-F 2 "foostan-kbd:CherryMX_Choc_1u" H 1350 1050 50  0001 C CNN
+F 2 "custom:CherryMX_Choc_1u" H 1350 1050 50  0001 C CNN
 F 3 "" H 1350 1050 50  0001 C CNN
 	1    1350 850
@@
 F 0 "SW19" H 2700 1935 50  0000 C CNN
 F 1 "SW_Push" H 2700 1844 50  0000 C CNN
-F 2 "foostan-kbd:CherryMX_Choc_1u" H 2700 1850 50  0001 C CNN
+F 2 "custom:CherryMX_Choc_1u" H 2700 1850 50  0001 C CNN
 F 3 "" H 2700 1850 50  0001 C CNN
 	1    2700 1650
@@
 F 0 "SW18" H 2700 1535 50  0000 C CNN
 F 1 "SW_Push" H 2700 1444 50  0000 C CNN
-F 2 "foostan-kbd:CherryMX_Choc_1u" H 2700 1450 50  0001 C CNN
+F 2 "custom:CherryMX_Choc_1u" H 2700 1450 50  0001 C CNN
 F 3 "" H 2700 1450 50  0001 C CNN
 	1    2700 1250
@@
 F 0 "SW17" H 2700 1135 50  0000 C CNN
 F 1 "SW_Push" H 2700 1044 50  0000 C CNN
-F 2 "foostan-kbd:CherryMX_Choc_1u" H 2700 1050 50  0001 C CNN
+F 2 "custom:CherryMX_Choc_1u" H 2700 1050 50  0001 C CNN
 F 3 "" H 2700 1050 50  0001 C CNN
 	1    2700 850
@@
 F 0 "SW14" H 1350 5585 50  0000 C CNN
 F 1 "SW_Push" H 1350 5494 50  0000 C CNN
-F 2 "foostan-kbd:CherryMX_Choc_1u" H 1350 5500 50  0001 C CNN
+F 2 "custom:CherryMX_Choc_1u" H 1350 5500 50  0001 C CNN
 F 3 "" H 1350 5500 50  0001 C CNN
 	1    1350 5300
@@
 F 0 "SW15" H 1350 5985 50  0000 C CNN
 F 1 "SW_Push" H 1350 5894 50  0000 C CNN
-F 2 "foostan-kbd:CherryMX_Choc_1u" H 1350 5900 50  0001 C CNN
+F 2 "custom:CherryMX_Choc_1u" H 1350 5900 50  0001 C CNN
 F 3 "" H 1350 5900 50  0001 C CNN
 	1    1350 5700
@@
 F 0 "SW13" H 1350 5185 50  0000 C CNN
 F 1 "SW_Push" H 1350 5094 50  0000 C CNN
-F 2 "foostan-kbd:CherryMX_Choc_1u" H 1350 5100 50  0001 C CNN
+F 2 "custom:CherryMX_Choc_1u" H 1350 5100 50  0001 C CNN
 F 3 "" H 1350 5100 50  0001 C CNN
 	1    1350 4900
@@
 F 0 "SW12" H 1350 4785 50  0000 C CNN
 F 1 "SW_Push" H 1350 4694 50  0000 C CNN
-F 2 "foostan-kbd:CherryMX_Choc_1u" H 1350 4700 50  0001 C CNN
+F 2 "custom:CherryMX_Choc_1u" H 1350 4700 50  0001 C CNN
 F 3 "" H 1350 4700 50  0001 C CNN
 	1    1350 4500

Commit message: Fix LDO
Parts:
- U2: symbol Regulator_Linear:LM3480-3.3 -> Regulator_Linear:MCP1703A-3302_SOT23
Connections:
- net 3.3V: now also U2.2 (VO); no longer U2.1 (VO)
- net 5V: now also U2.3 (VI); no longer U2.2 (VI)
- net GND: now also U2.1 (GND); no longer U2.3 (GND)
Changed lines of the file:
@@
 Connection ~ 4450 1600
 $Comp
-L Regulator_Linear:LM3480-3.3 U2
+L Regulator_Linear:MCP1703A-3302_SOT23 U2
 U 1 1 5DED53E7
 P 8250 900
