File: pcb/kicad/left/left.sch (KiCad schematic (older format))
At the start: 61 parts, among them J1 USB_C_Receptacle_USB2.0, J2 AudioJack4, J3 Conn_01x12_Male, SW1 BOOT, SW10 SW_Push, SW12 SW_Push, SW13 SW_Push, SW14 SW_Push, SW15 SW_Push, SW17 SW_Push, SW18 SW_Push, SW19 SW_Push, SW2 RESET, SW21 SW_Push, SW22 SW_Push, SW23 SW_Push, SW24 SW_Push, SW3 SW_Push, SW31 SW_Push, SW32 SW_Push, SW33 SW_Push, SW34 SW_Push, SW4 SW_Push, SW5 SW_Push, SW7 SW_Push, SW8 SW_Push, SW9 SW_Push, U1 STM32, U2 LDO

Commit message: Small changes for left manufactured SMT
Parts:
- J1: LCSC C165948 -> C136423
Changed lines of the file:
@@
 F 2 "kicad-usb:USB_C_Receptacle_HRO_TYPE-C-31-M-12" H 10900 1500 50  0001 C CNN
 F 3 "https://www.usb.org/sites/default/files/documents/usb_type-c.zip" H 10900 1500 50  0001 C CNN
-F 4 "C165948" H 10750 1500 50  0001 C CNN "LCSC"
+F 4 "C136423" H 10750 1500 50  0001 C CNN "LCSC"
 	1    10750 1500
 	-1   0    0    -1
