File: pcb/kicad/left/_autosave-left.sch (KiCad schematic (older format))
At the start: 61 parts, among them J1 USB_C_Receptacle_USB2.0, J2 AudioJack4, J3 Conn_01x12_Male, SW1 BOOT, SW10 SW_Push, SW12 SW_Push, SW13 SW_Push, SW14 SW_Push, SW15 SW_Push, SW17 SW_Push, SW18 SW_Push, SW19 SW_Push, SW2 RESET, SW21 SW_Push, SW22 SW_Push, SW23 SW_Push, SW24 SW_Push, SW3 SW_Push, SW31 SW_Push, SW32 SW_Push, SW33 SW_Push, SW34 SW_Push, SW4 SW_Push, SW5 SW_Push, SW7 SW_Push, SW8 SW_Push, SW9 SW_Push, U1 STM32, U2 LDO

Commit message: Some try at STM assembly (clearly not yet ready)
Parts:
- C1, C2, C3, C4, C5: LCSC C60474 -> C49678
- C6, C7: LCSC C282732 -> C28323
- D10, D11, D12, D14, D15, D16, D17, D19, D20, D21, D23, D24, D25, D26, D33, D34, D35, D36, D5, D6, D7, D9: LCSC C908249 -> C2128
- R1, R6, R7: LCSC C269748 -> C27834
- U2: LCSC C347376 -> C5446
Changed lines of the file:
@@
 F 2 "Capacitor_SMD:C_0805_2012Metric_Pad1.15x1.40mm_HandSolder" H 5738 600 50  0001 C CNN
 F 3 "~" H 5700 750 50  0001 C CNN
-F 4 "C60474" H 5700 750 50  0001 C CNN "LCSC"
+F 4 " C49678" H 5700 750 50  0001 C CNN "LCSC"
 	1    5700 750
 	1    0    0    -1
@@
 F 2 "Capacitor_SMD:C_0805_2012Metric_Pad1.15x1.40mm_HandSolder" H 6188 600 50  0001 C CNN
 F 3 "~" H 6150 750 50  0001 C CNN
-F 4 "C60474" H 6150 750 50  0001 C CNN "LCSC"
+F 4 " C49678" H 6150 750 50  0001 C CNN "LCSC"
 	1    6150 750
 	1    0    0    -1
@@
 F 2 "Capacitor_SMD:C_0805_2012Metric_Pad1.15x1.40mm_HandSolder" H 6638 600 50  0001 C CNN
 F 3 "~" H 6600 750 50  0001 C CNN
-F 4 "C60474" H 6600 750 50  0001 C CNN "LCSC"
+F 4 " C49678" H 6600 750 50  0001 C CNN "LCSC"
 	1    6600 750
 	1    0    0    -1
@@
 F 2 "Capacitor_SMD:C_0805_2012Metric_Pad1.15x1.40mm_HandSolder" H 7138 600 50  0001 C CNN
 F 3 "~" H 7100 750 50  0001 C CNN
-F 4 "C60474" H 7100 750 50  0001 C CNN "LCSC"
+F 4 " C49678" H 7100 750 50  0001 C CNN "LCSC"
 	1    7100 750
 	1    0    0    -1
@@
 F 2 "Capacitor_SMD:C_0805_2012Metric_Pad1.15x1.40mm_HandSolder" H 8688 600 50  0001 C CNN
 F 3 "~" H 8650 750 50  0001 C CNN
-F 4 "C282732" H 8650 750 50  0001 C CNN "LCSC"
+F 4 "C28323" H 8650 750 50  0001 C CNN "LCSC"
 	1    8650 750
 	1    0    0    -1
@@
 F 2 "Capacitor_SMD:C_0805_2012Metric_Pad1.15x1.40mm_HandSolder" H 5088 1000 50  0001 C CNN
 F 3 "~" H 5050 1150 50  0001 C CNN
-F 4 "C60474" H 5050 1150 50  0001 C CNN "LCSC"
+F 4 " C49678" H 5050 1150 50  0001 C CNN "LCSC"
 	1    5050 1150
 	1    0    0    -1
@@
 F 2 "Resistor_SMD:R_0805_2012Metric_Pad1.15x1.40mm_HandSolder" V 4380 1750 50  0001 C CNN
 F 3 "~" H 4450 1750 50  0001 C CNN
-F 4 "C269748" H 4450 1750 50  0001 C CNN "LCSC"
+F 4 "C27834" H 4450 1750 50  0001 C CNN "LCSC"
 	1    4450 1750
 	1    0    0    -1
@@
 F 2 "Package_TO_SOT_SMD:SOT-23" H 8250 1125 50  0001 C CIN
 F 3 "http://www.ti.com/lit/ds/symlink/lm3480.pdf" H 8250 900 50  0001 C CNN
-F 4 "C347376" H 8250 900 50  0001 C CNN "LCSC"
+F 4 "C5446" H 8250 900 50  0001 C CNN "LCSC"
 	1    8250 900
 	-1   0    0    1
@@
 F 2 "Resistor_SMD:R_0805_2012Metric_Pad1.15x1.40mm_HandSolder" V 9930 1100 50  0001 C CNN
 F 3 "~" H 10000 1100 50  0001 C CNN
-F 4 "C269748" H 10000 1100 50  0001 C CNN "LCSC"
+F 4 "C27834" H 10000 1100 50  0001 C CNN "LCSC"
 	1    10000 1100
 	0    1    1    0
@@
 F 2 "Resistor_SMD:R_0805_2012Metric_Pad1.15x1.40mm_HandSolder" V 9430 1200 50  0001 C CNN
 F 3 "~" H 9500 1200 50  0001 C CNN
-F 4 "C269748" H 9500 1200 50  0001 C CNN "LCSC"
+F 4 "C27834" H 9500 1200 50  0001 C CNN "LCSC"
 	1    9500 1200
 	0    1    -1   0
@@
 F 2 "Capacitor_SMD:C_0805_2012Metric_Pad1.15x1.40mm_HandSolder" H 7638 600 50  0001 C CNN
 F 3 "~" H 7600 750 50  0001 C CNN
-F 4 "C282732" H 7600 750 50  0001 C CNN "LCSC"
+F 4 "C28323" H 7600 750 50  0001 C CNN "LCSC"
 	1    7600 750
 	1    0    0    -1
@@
 F 2 "Diode_SMD:D_SOD-323_HandSoldering" H 1000 3350 50  0001 C CNN
 F 3 "~" H 1000 3350 50  0001 C CNN
-F 4 "C908249" H 1000 3350 50  0001 C CNN "LCSC"
+F 4 "C2128" H 1000 3350 50  0001 C CNN "LCSC"
 	1    1000 3350
 	1    0    0    -1
@@
 F 2 "Diode_SMD:D_SOD-323_HandSoldering" H 1000 3750 50  0001 C CNN
 F 3 "~" H 1000 3750 50  0001 C CNN
-F 4 "C908249" H 1000 3750 50  0001 C CNN "LCSC"
+F 4 "C2128" H 1000 3750 50  0001 C CNN "LCSC"
 	1    1000 3750
 	1    0    0    -1
@@
 F 2 "Diode_SMD:D_SOD-323_HandSoldering" H 1000 2950 50  0001 C CNN
 F 3 "~" H 1000 2950 50  0001 C CNN
-F 4 "C908249" H 1000 2950 50  0001 C CNN "LCSC"
+F 4 "C2128" H 1000 2950 50  0001 C CNN "LCSC"
 	1    1000 2950
 	1    0    0    -1
@@
 F 2 "Diode_SMD:D_SOD-323_HandSoldering" H 1000 2550 50  0001 C CNN
 F 3 "~" H 1000 2550 50  0001 C CNN
-F 4 "C908249" H 1000 2550 50  0001 C CNN "LCSC"
+F 4 "C2128" H 1000 2550 50  0001 C CNN "LCSC"
 	1    1000 2550
 	1    0    0    -1
@@
 F 2 "Diode_SMD:D_SOD-323_HandSoldering" H 2350 3350 50  0001 C CNN
 F 3 "~" H 2350 3350 50  0001 C CNN
-F 4 "C908249" H 2350 3350 50  0001 C CNN "LCSC"
+F 4 "C2128" H 2350 3350 50  0001 C CNN "LCSC"
 	1    2350 3350
 	1    0    0    -1
@@
 F 2 "Diode_SMD:D_SOD-323_HandSoldering" H 2350 3750 50  0001 C CNN
 F 3 "~" H 2350 3750 50  0001 C CNN
-F 4 "C908249" H 2350 3750 50  0001 C CNN "LCSC"
+F 4 "C2128" H 2350 3750 50  0001 C CNN "LCSC"
 	1    2350 3750
 	1    0    0    -1
@@
 F 2 "Diode_SMD:D_SOD-323_HandSoldering" H 2350 2950 50  0001 C CNN
 F 3 "~" H 2350 2950 50  0001 C CNN
-F 4 "C908249" H 2350 2950 50  0001 C CNN "LCSC"
+F 4 "C2128" H 2350 2950 50  0001 C CNN "LCSC"
 	1    2350 2950
 	1    0    0    -1
@@
 F 2 "Diode_SMD:D_SOD-323_HandSoldering" H 2350 2550 50  0001 C CNN
 F 3 "~" H 2350 2550 50  0001 C CNN
-F 4 "C908249" H 2350 2550 50  0001 C CNN "LCSC"
+F 4 "C2128" H 2350 2550 50  0001 C CNN "LCSC"
 	1    2350 2550
 	1    0    0    -1
@@
 F 2 "Diode_SMD:D_SOD-323_HandSoldering" H 3700 3350 50  0001 C CNN
 F 3 "~" H 3700 3350 50  0001 C CNN
-F 4 "C908249" H 3700 3350 50  0001 C CNN "LCSC"
+F 4 "C2128" H 3700 3350 50  0001 C CNN "LCSC"
 	1    3700 3350
 	1    0    0    -1
@@
 F 2 "Diode_SMD:D_SOD-323_HandSoldering" H 3700 3750 50  0001 C CNN
 F 3 "~" H 3700 3750 50  0001 C CNN
-F 4 "C908249" H 3700 3750 50  0001 C CNN "LCSC"
+F 4 "C2128" H 3700 3750 50  0001 C CNN "LCSC"
 	1    3700 3750
 	1    0    0    -1
@@
 F 2 "Diode_SMD:D_SOD-323_HandSoldering" H 3700 2950 50  0001 C CNN
 F 3 "~" H 3700 2950 50  0001 C CNN
-F 4 "C908249" H 3700 2950 50  0001 C CNN "LCSC"
+F 4 "C2128" H 3700 2950 50  0001 C CNN "LCSC"
 	1    3700 2950
 	1    0    0    -1
@@
 F 2 "Diode_SMD:D_SOD-323_HandSoldering" H 3700 2550 50  0001 C CNN
 F 3 "~" H 3700 2550 50  0001 C CNN
-F 4 "C908249" H 3700 2550 50  0001 C CNN "LCSC"
+F 4 "C2128" H 3700 2550 50  0001 C CNN "LCSC"
 	1    3700 2550
 	1    0    0    -1
@@
 F 2 "Diode_SMD:D_SOD-323_HandSoldering" H 1000 1650 50  0001 C CNN
 F 3 "~" H 1000 1650 50  0001 C CNN
-F 4 "C908249" H 1000 1650 50  0001 C CNN "LCSC"
+F 4 "C2128" H 1000 1650 50  0001 C CNN "LCSC"
 	1    1000 1650
 	1    0    0    -1
@@
 F 2 "Diode_SMD:D_SOD-323_HandSoldering" H 1000 1250 50  0001 C CNN
 F 3 "~" H 1000 1250 50  0001 C CNN
-F 4 "C908249" H 1000 1250 50  0001 C CNN "LCSC"
+F 4 "C2128" H 1000 1250 50  0001 C CNN "LCSC"
 	1    1000 1250
 	1    0    0    -1
@@
 F 2 "Diode_SMD:D_SOD-323_HandSoldering" H 1000 850 50  0001 C CNN
 F 3 "~" H 1000 850 50  0001 C CNN
-F 4 "C908249" H 1000 850 50  0001 C CNN "LCSC"
+F 4 "C2128" H 1000 850 50  0001 C CNN "LCSC"
 	1    1000 850
 	1    0    0    -1
@@
 F 2 "Diode_SMD:D_SOD-323_HandSoldering" H 2350 1650 50  0001 C CNN
 F 3 "~" H 2350 1650 50  0001 C CNN
-F 4 "C908249" H 2350 1650 50  0001 C CNN "LCSC"
+F 4 "C2128" H 2350 1650 50  0001 C CNN "LCSC"
 	1    2350 1650
 	1    0    0    -1
@@
 F 2 "Diode_SMD:D_SOD-323_HandSoldering" H 2350 1250 50  0001 C CNN
 F 3 "~" H 2350 1250 50  0001 C CNN
-F 4 "C908249" H 2350 1250 50  0001 C CNN "LCSC"
+F 4 "C2128" H 2350 1250 50  0001 C CNN "LCSC"
 	1    2350 1250
 	1    0    0    -1
@@
 F 2 "Diode_SMD:D_SOD-323_HandSoldering" H 2350 850 50  0001 C CNN
 F 3 "~" H 2350 850 50  0001 C CNN
-F 4 "C908249" H 2350 850 50  0001 C CNN "LCSC"
+F 4 "C2128" H 2350 850 50  0001 C CNN "LCSC"
 	1    2350 850
 	1    0    0    -1
@@
 F 2 "Diode_SMD:D_SOD-323_HandSoldering" H 1000 5300 50  0001 C CNN
 F 3 "~" H 1000 5300 50  0001 C CNN
-F 4 "C908249" H 1000 5300 50  0001 C CNN "LCSC"
+F 4 "C2128" H 1000 5300 50  0001 C CNN "LCSC"
 	1    1000 5300
 	1    0    0    -1
@@
 F 2 "Diode_SMD:D_SOD-323_HandSoldering" H 1000 5700 50  0001 C CNN
 F 3 "~" H 1000 5700 50  0001 C CNN
-F 4 "C908249" H 1000 5700 50  0001 C CNN "LCSC"
+F 4 "C2128" H 1000 5700 50  0001 C CNN "LCSC"
 	1    1000 5700
 	1    0    0    -1
@@
 F 2 "Diode_SMD:D_SOD-323_HandSoldering" H 1000 4900 50  0001 C CNN
 F 3 "~" H 1000 4900 50  0001 C CNN
-F 4 "C908249" H 1000 4900 50  0001 C CNN "LCSC"
+F 4 "C2128" H 1000 4900 50  0001 C CNN "LCSC"
 	1    1000 4900
 	1    0    0    -1
@@
 F 2 "Diode_SMD:D_SOD-323_HandSoldering" H 1000 4500 50  0001 C CNN
 F 3 "~" H 1000 4500 50  0001 C CNN
-F 4 "C908249" H 1000 4500 50  0001 C CNN "LCSC"
+F 4 "C2128" H 1000 4500 50  0001 C CNN "LCSC"
 	1    1000 4500
 	1    0    0    -1
